Commit message: URDF edit for correct motor input, HuboLCMType simplified.

File: matlab-model/urdf/hubo_base_link.urdf (robot description, URDF)
Before this commit: robot hubo2, 60 links, 59 joints
Links:
- removed link Body_LAP
- removed link Body_LAR
- removed link Body_LEB
- removed link Body_LHP
- removed link Body_LHR
- removed link Body_LHY
- removed link Body_LKN
- removed link Body_LSP
- removed link Body_LSR
- removed link Body_LSY
- removed link Body_LWP
- removed link Body_LWY
- removed link Body_RAP
- removed link Body_RAR
- removed link Body_REB
- removed link Body_RHP
- removed link Body_RHR
- removed link Body_RHY
- removed link Body_RKN
- removed link Body_RSP
- removed link Body_RSR
- removed link Body_RSY
- removed link Body_RWP
- removed link Body_RWY
- added link Body_LeftAnklePitch, mass 1.63501; collision mesh filename=./meshes/Body_LAP.stl; visual mesh filename=./meshes/Body_LAP.stl
- added link Body_LeftAnkleRoll, mass 1.20318; collision mesh filename=./meshes/Body_LAR.stl; visual mesh filename=./meshes/Body_LAR.stl
- added link Body_LeftElbowPitch, mass 0.44094; collision mesh filename=./meshes/Body_LEB.stl; visual mesh filename=./meshes/Body_LEB.stl
- added link Body_LeftHipPitch, mass 2.8201; collision mesh filename=./meshes/Body_LHP.stl; visual mesh filename=./meshes/Body_LHP.stl
- added link Body_LeftHipRoll, mass 1.93266; collision mesh filename=./meshes/Body_LHR.stl; visual mesh filename=./meshes/Body_LHR.stl
- added link Body_LeftHipYaw, mass 0.826125; collision mesh filename=./meshes/Body_LHY.stl; visual mesh filename=./meshes/Body_LHY.stl
- added link Body_LeftKneePitch, mass 1.80912; collision mesh filename=./meshes/Body_LKN.stl; visual mesh filename=./meshes/Body_LKN_vis.dae
- added link Body_LeftShoulderPitch, mass 0.646655; collision mesh filename=./meshes/Body_LSP.stl; visual mesh filename=./meshes/Body_LSP.stl
- added link Body_LeftShoulderRoll, mass 0.413368; collision mesh filename=./meshes/Body_LSR.stl; visual mesh filename=./meshes/Body_LSR.stl
- added link Body_LeftShoulderYaw, mass 1.15461; collision mesh filename=./meshes/Body_LSY.stl; visual mesh filename=./meshes/Body_LSY_vis.dae
- added link Body_LeftWristPitch, mass 0.164393; collision mesh filename=./meshes/Body_LWP.stl; visual mesh filename=./meshes/Body_LWP_vis.dae
- added link Body_LeftWristYaw, mass 0.537738; collision mesh filename=./meshes/Body_LWY.stl; visual mesh filename=./meshes/Body_LWY_vis.dae
- added link Body_RightAnklePitch, mass 1.63501; collision mesh filename=./meshes/Body_RAP.stl; visual mesh filename=./meshes/Body_RAP_vis.dae
- added link Body_RightAnkleRoll, mass 1.20318; collision mesh filename=./meshes/Body_RAR.stl; visual mesh filename=./meshes/Body_RAR_vis.dae
- added link Body_RightElbowPitch, mass 0.44094; collision mesh filename=./meshes/Body_REB.stl; visual mesh filename=./meshes/Body_REB_vis.dae
- added link Body_RightHipPitch, mass 2.8201; collision mesh filename=./meshes/Body_RHP.stl; visual mesh filename=./meshes/Body_RHP_vis.dae
- added link Body_RightHipRoll, mass 1.93266; collision mesh filename=./meshes/Body_RHR.stl; visual mesh filename=./meshes/Body_RHR_vis.dae
- added link Body_RightHipYaw, mass 0.826125; collision mesh filename=./meshes/Body_RHY.stl; visual mesh filename=./meshes/Body_RHY_vis.dae
- added link Body_RightKneePitch, mass 1.80912; collision mesh filename=./meshes/Body_RKN.stl; visual mesh filename=./meshes/Body_RKN_vis.dae
- added link Body_RightShoulderPitch, mass 0.646655; collision mesh filename=./meshes/Body_RSP.stl; visual mesh filename=./meshes/Body_RSP_vis.dae
- added link Body_RightShoulderRoll, mass 0.413368; collision mesh filename=./meshes/Body_RSR.stl; visual mesh filename=./meshes/Body_RSR_vis.dae
- added link Body_RightShoulderYaw, mass 1.15461; collision mesh filename=./meshes/Body_RSY.stl; visual mesh filename=./meshes/Body_RSY_vis.dae
- added link Body_RightWristPitch, mass 0.164393; collision mesh filename=./meshes/Body_RWP.stl; visual mesh filename=./meshes/Body_RWP_vis.dae
- added link Body_RightWristYaw, mass 0.537738; collision mesh filename=./meshes/Body_RWY.stl; visual mesh filename=./meshes/Body_RWY_vis.dae
Joints:
- removed joint HNP
- removed joint HNR
- removed joint LAP
- removed joint LAR
- removed joint LEB
- removed joint LHP
- removed joint LHR
- removed joint LHY
- removed joint LKN
- removed joint LSP
- removed joint LSR
- removed joint LSY
- removed joint LWP
- removed joint LWY
- removed joint NKY
- removed joint RAP
- removed joint RAR
- removed joint REB
- removed joint RHP
- removed joint RHR
- removed joint RHY
- removed joint RKN
- removed joint RSP
- removed joint RSR
- removed joint RSY
- removed joint RWP
- removed joint RWY
- removed joint WST
- removed joint leftIndexKnuckle1
- removed joint leftMiddleKnuckle1
- removed joint leftPinkyKnuckle1
- removed joint leftRingKnuckle1
- removed joint leftThumbKnuckle1
- removed joint rightIndexKnuckle1
- removed joint rightMiddleKnuckle1
- removed joint rightPinkyKnuckle1
- removed joint rightRingKnuckle1
- removed joint rightThumbKnuckle1
- added joint LeftAnklePitch: type revolute, parent Body_LeftKneePitch, child Body_LeftAnklePitch, origin xyz=7.20248e-06 0.0247555 -0.279942 rpy=0 -0 0, axis 0 1 0, limit lower=-1.29154 upper=1.69297 effort=10.0 velocity=1.0
- added joint LeftAnkleRoll: type revolute, parent Body_LeftAnklePitch, child Body_LeftAnkleRoll, origin xyz=0.0711787 -0.0466006 -1.04e-10 rpy=0 -0 0, axis 1 0 0, limit lower=-0.191986 upper=0.191986 effort=10.0 velocity=1.0
- added joint LeftElbowPitch: type revolute, parent Body_LeftShoulderYaw, child Body_LeftElbowPitch, origin xyz=0.0219936 -0.018 -0.157505 rpy=0 -0 0, axis 0 1 0, limit lower=-2.49582 upper=0.0698132 effort=10.0 velocity=1.0
- added joint LeftFinger1: type revolute, parent Body_LeftWristPitch, child leftThumbProximal, origin xyz=0.0208959 0.00192069 -0.060952 rpy=1.5708 -0.785398 -1.5708, axis 0 0 -1, limit lower=-3.14 upper=3.14 effort=10.0 velocity=1.0
- added joint LeftFinger2: type revolute, parent Body_LeftWristPitch, child leftIndexProximal, origin xyz=0.0289159 0.0298617 -0.088883 rpy=1.5708 0.785398 1.5708, axis 0 0 -1, limit lower=-3.14 upper=3.14 effort=10.0 velocity=1.0
- added joint LeftFinger3: type revolute, parent Body_LeftWristPitch, child leftMiddleProximal, origin xyz=0.00993585 0.0298617 -0.088883 rpy=1.5708 0.785398 1.5708, axis 0 0 -1, limit lower=-3.14 upper=3.14 effort=10.0 velocity=1.0
- added joint LeftFinger4: type revolute, parent Body_LeftWristPitch, child leftRingProximal, origin xyz=-0.00910415 0.0298617 -0.088883 rpy=1.5708 0.785398 1.5708, axis 0 0 -1, limit lower=-3.14 upper=3.14 effort=10.0 velocity=1.0
- added joint LeftFinger5: type revolute, parent Body_LeftWristPitch, child leftPinkyProximal, origin xyz=-0.0281041 0.0298617 -0.088883 rpy=1.5708 0.785398 1.5708, axis 0 0 -1, limit lower=-3.14 upper=3.14 effort=10.0 velocity=1.0
- added joint LeftHipPitch: type revolute, parent Body_LeftHipRoll, child Body_LeftHipPitch, origin xyz=-0.0529074 0.0655748 9.99159e-05 rpy=0 -0 0, axis 0 1 0, limit lower=-1.48353 upper=1.6057 effort=10.0 velocity=1.0
- added joint LeftHipRoll: type revolute, parent Body_LeftHipYaw, child Body_LeftHipRoll, origin xyz=0.0520001 1.50498e-06 -0.091004 rpy=0 -0 0, axis 1 0 0, limit lower=-0.488692 upper=0.488692 effort=10.0 velocity=1.0
- added joint LeftHipYaw: type revolute, parent Body_Hip, child Body_LeftHipYaw, origin xyz=0.000125136 0.0885155 -0.0764689 rpy=0 -0 0, axis 0 0 1, limit lower=-1.5708 upper=1.5708 effort=10.0 velocity=1.0
- added joint LeftKneePitch: type revolute, parent Body_LeftHipPitch, child Body_LeftKneePitch, origin xyz=0.000766364 -0.0445011 -0.280007 rpy=0 -0 0, axis 0 1 0, limit lower=-0.0698132 upper=2.60054 effort=10.0 velocity=1.0
- added joint LeftShoulderPitch: type revolute, parent Body_Torso, child Body_LeftShoulderPitch, origin xyz=0.0122581 0.143973 1.0486356 rpy=0 -0 0, axis 0 1 0, limit lower=-3.14158 upper=3.14158 effort=10.0 velocity=1.0
- added joint LeftShoulderRoll: type revolute, parent Body_LeftShoulderPitch, child Body_LeftShoulderRoll, origin xyz=0.0269 0.072 0 rpy=0 -0 0, axis 1 0 0, limit lower=0 upper=3.14158 effort=10.0 velocity=1.0
- added joint LeftShoulderYaw: type revolute, parent Body_LeftShoulderRoll, child Body_LeftShoulderYaw, origin xyz=-0.0269 -0.000166249 -0.0245 rpy=0 -0 0, axis 0 0 1, limit lower=-3.14158 upper=3.14158 effort=10.0 velocity=1.0
- added joint LeftWristPitch: type revolute, parent Body_LeftWristYaw, child Body_LeftWristPitch, origin xyz=1.72973e-06 -0.00872953 -0.05255 rpy=0 -0 0, axis 0 1 0, limit lower=-1.64061 upper=1.01229 effort=10.0 velocity=1.0
- added joint LeftWristYaw: type revolute, parent Body_LeftElbowPitch, child Body_LeftWristYaw, origin xyz=-0.0219906 0.018 -0.111408 rpy=0 -0 0, axis 0 0 1, limit lower=-3.14158 upper=3.14158 effort=10.0 velocity=1.0
- added joint Neck1: type revolute, parent Body_Neck, child Body_Head_Empty, origin xyz=-0.0014665 0.0024526 0.0876725 rpy=0 -0 0, axis 0 1 0, limit lower=-0.523599 upper=0.523599 effort=10.0 velocity=1.0
- added joint Neck2: type revolute, parent Body_Head_Empty, child Body_Head, origin xyz=0 0 0 rpy=0 -0 0, axis 1 0 0, limit lower=-0.523599 upper=0.523599 effort=10.0 velocity=1.0
- added joint NeckYaw: type revolute, parent Body_Torso, child Body_Neck, origin xyz=0.0137246 0.0 1.1092625 rpy=0 -0 0, axis 0 0 1, limit lower=-1.5 upper=1.5 effort=10.0 velocity=1.0
- added joint RightAnklePitch: type revolute, parent Body_RightKneePitch, child Body_RightAnklePitch, origin xyz=7.20248e-06 -0.0247555 -0.279942 rpy=0 -0 0, axis 0 1 0, limit lower=-1.29154 upper=1.69297 effort=10.0 velocity=1.0
- added joint RightAnkleRoll: type revolute, parent Body_RightAnklePitch, child Body_RightAnkleRoll, origin xyz=0.0711787 0.0466006 -1.04e-10 rpy=0 -0 0, axis 1 0 0, limit lower=-0.191986 upper=0.191986 effort=10.0 velocity=1.0
- added joint RightElbowPitch: type revolute, parent Body_RightShoulderYaw, child Body_RightElbowPitch, origin xyz=0.0219936 0.018 -0.157505 rpy=0 -0 0, axis 0 1 0, limit lower=-2.49582 upper=0.0698132 effort=10.0 velocity=1.0
- added joint RightFinger1: type revolute, parent Body_RightWristPitch, child rightThumbProximal, origin xyz=0.0208959 -0.00192069 -0.060952 rpy=1.5708 -0.785398 1.5708, axis 0 0 -1, limit lower=0 upper=1.57 effort=10.0 velocity=1.0
- added joint RightFinger2: type revolute, parent Body_RightWristPitch, child rightIndexProximal, origin xyz=0.0289159 -0.0298617 -0.088883 rpy=1.5708 0.785398 -1.5708, axis 0 0 -1, limit lower=0 upper=1.57 effort=10.0 velocity=1.0
- added joint RightFinger3: type revolute, parent Body_RightWristPitch, child rightMiddleProximal, origin xyz=0.00993585 -0.0298617 -0.088883 rpy=1.5708 0.785398 -1.5708, axis 0 0 -1, limit lower=0 upper=1.57 effort=10.0 velocity=1.0
- added joint RightFinger4: type revolute, parent Body_RightWristPitch, child rightRingProximal, origin xyz=-0.00910415 -0.0298617 -0.088883 rpy=1.5708 0.785398 -1.5708, axis 0 0 -1, limit lower=0 upper=1.57 effort=10.0 velocity=1.0
- added joint RightFinger5: type revolute, parent Body_RightWristPitch, child rightPinkyProximal, origin xyz=-0.0281041 -0.0298617 -0.088883 rpy=1.5708 0.785398 -1.5708, axis 0 0 -1, limit lower=0 upper=1.57 effort=10.0 velocity=1.0
- added joint RightHipPitch: type revolute, parent Body_RightHipRoll, child Body_RightHipPitch, origin xyz=-0.0529074 -0.0655748 9.99159e-05 rpy=0 -0 0, axis 0 1 0, limit lower=-1.48353 upper=1.6057 effort=10.0 velocity=1.0
- added joint RightHipRoll: type revolute, parent Body_RightHipYaw, child Body_RightHipRoll, origin xyz=0.0520001 7.3455e-05 -0.091004 rpy=0 -0 0, axis 1 0 0, limit lower=-0.488692 upper=0.488692 effort=10.0 velocity=1.0
- added joint RightHipYaw: type revolute, parent Body_Hip, child Body_RightHipYaw, origin xyz=0.000125136 -0.0884999 -0.0764689 rpy=0 -0 0, axis 0 0 1, limit lower=-1.5708 upper=1.5708 effort=10.0 velocity=1.0
- added joint RightKneePitch: type revolute, parent Body_RightHipPitch, child Body_RightKneePitch, origin xyz=0.000766364 0.0445011 -0.280007 rpy=0 -0 0, axis 0 1 0, limit lower=-0.0698132 upper=2.60054 effort=10.0 velocity=1.0
- added joint RightShoulderPitch: type revolute, parent Body_Torso, child Body_RightShoulderPitch, origin xyz=0.0122581 -0.139027 1.0486356 rpy=0 -0 0, axis 0 1 0, limit lower=-3.14158 upper=3.14158 effort=10.0 velocity=1.0
- added joint RightShoulderRoll: type revolute, parent Body_RightShoulderPitch, child Body_RightShoulderRoll, origin xyz=0.0269 -0.072 0 rpy=0 -0 0, axis 1 0 0, limit lower=-3.14158 upper=0 effort=10.0 velocity=1.0
- added joint RightShoulderYaw: type revolute, parent Body_RightShoulderRoll, child Body_RightShoulderYaw, origin xyz=-0.0269 0 -0.0245 rpy=0 -0 0, axis 0 0 1, limit lower=-3.14158 upper=3.14158 effort=10.0 velocity=1.0
- added joint RightWristPitch: type revolute, parent Body_RightWristYaw, child Body_RightWristPitch, origin xyz=1.72973e-06 0.01 -0.05255 rpy=0 -0 0, axis 0 1 0, limit lower=-1.64061 upper=1.01229 effort=10.0 velocity=1.0
- added joint RightWristYaw: type revolute, parent Body_RightElbowPitch, child Body_RightWristYaw, origin xyz=-0.0219906 -0.018 -0.111408 rpy=0 -0 0, axis 0 0 1, limit lower=-3.14158 upper=3.14158 effort=10.0 velocity=1.0
- added joint TrunkYaw: type revolute, parent Body_Torso, child Body_Hip, origin xyz=0.0122662 0.00245974 0.84738 rpy=0 -0 0, axis 0 0 -1, limit lower=-3.14158 upper=3.14158 effort=10.0 velocity=1.0
